Commit message: Add world sdf, navigation, and arm control nodes
- Add Gazebo world (SDF) with two-room house layout and furniture
- Add nav_node for waypoint-following navigation with LiDAR obstacle avoidance
- Add arm_init_node to publish a tucked arm pose on spawn
- Add ROS 2–Gazebo bridge config for sensors, drive, and arm joints
- Add sim launch file to bring up Gazebo, bridge, and all nodes

File: home-tidying-robot/urdf/home-tidying-robot.urdf.xacro (robot description, xacro)
@@ -69,4 +69,14 @@
             <cylinder radius="0.075" length="0.04"/>
         </geometry>
+        <surface>
+        <friction>
+            <ode>
+            <mu>1.0</mu>
+            <mu2>0.8</mu2>
+            <kp>1000000</kp>
+            <kd>100</kd>
+            </ode>
+        </friction>
+        </surface>
         </collision>
         <inertial>
@@ -96,4 +106,14 @@
             <cylinder radius="0.075" length="0.04"/>
         </geometry>
+        <surface>
+        <friction>
+            <ode>
+            <mu>1.0</mu>
+            <mu2>0.8</mu2>
+            <kp>1000000</kp>
+            <kd>100</kd>
+            </ode>
+        </friction>
+        </surface>
         </collision>
         <inertial>
@@ -122,4 +142,14 @@
             <cylinder radius="0.075" length="0.04"/>
         </geometry>
+        <surface>
+        <friction>
+            <ode>
+            <mu>1.0</mu>
+            <mu2>0.8</mu2>
+            <kp>1000000</kp>
+            <kd>100</kd>
+            </ode>
+        </friction>
+        </surface>
         </collision>
         <inertial>
@@ -148,4 +178,14 @@
             <cylinder radius="0.075" length="0.04"/>
         </geometry>
+        <surface>
+        <friction>
+        <ode>
+            <mu>1.0</mu>
+            <mu2>0.8</mu2>
+            <kp>1000000</kp>
+            <kd>100</kd>
+        </ode>
+        </friction>
+        </surface>
         </collision>
         <inertial>
@@ -295,15 +335,15 @@
                ixy="0" ixz="0" iyz="0"/>
     </inertial>
-  </link>
-  <joint name="right_elbow_joint" type="revolute">
-    <parent link="right_upper_arm_link"/>
-    <child link="right_elbow_link"/>
-    <origin xyz="0 0 -0.28" rpy="0 0 0"/>
-    <axis xyz="0 1 0"/>
-    <limit lower="-2.356" upper="0.0" effort="20.0" velocity="1.5"/>
-    <dynamics damping="0.4" friction="0.08"/>
-  </joint>
-  <!-- Forearm -->
-  <link name="right_forearm_link">
+    </link>
+    <joint name="right_elbow_joint" type="revolute">
+        <parent link="right_upper_arm_link"/>
+        <child link="right_elbow_link"/>
+        <origin xyz="0 0 -0.28" rpy="0 0 0"/>
+        <axis xyz="0 1 0"/>
+        <limit lower="-2.356" upper="0.0" effort="20.0" velocity="1.5"/>
+        <dynamics damping="0.4" friction="0.08"/>
+    </joint>
+    <!-- Forearm -->
+    <link name="right_forearm_link">
     <visual>
       <geometry>
@@ -325,12 +365,12 @@
                ixy="0" ixz="0" iyz="0"/>
     </inertial>
-  </link>
-  <joint name="right_forearm_joint" type="fixed">
-    <parent link="right_elbow_link"/>
-    <child link="right_forearm_link"/>
-    <origin xyz="0 0 0" rpy="0 0 0"/>
-  </joint>
-  <!-- Wrist -->
-  <link name="right_wrist_link">
+    </link>
+    <joint name="right_forearm_joint" type="fixed">
+        <parent link="right_elbow_link"/>
+        <child link="right_forearm_link"/>
+        <origin xyz="0 0 0" rpy="0 0 0"/>
+    </joint>
+    <!-- Wrist -->
+    <link name="right_wrist_link">
     <visual>
       <geometry>
@@ -349,16 +389,16 @@
                ixy="0" ixz="0" iyz="0"/>
     </inertial>
-  </link>
-  <joint name="right_wrist_joint" type="revolute">
-    <parent link="right_forearm_link"/>
-    <child link="right_wrist_link"/>
-    <origin xyz="0 0 -0.26" rpy="0 0 0"/>
-    <axis xyz="0 1 0"/>
-    <limit lower="-1.571" upper="1.571" effort="10.0" velocity="2.0"/>
-    <dynamics damping="0.3" friction="0.05"/>
-  </joint>
-  <!-- Gripper (parallel-jaw style, modeled as two finger pads + a palm) -->
-  <!-- Palm -->
-  <link name="right_gripper_palm">
+    </link>
+    <joint name="right_wrist_joint" type="revolute">
+        <parent link="right_forearm_link"/>
+        <child link="right_wrist_link"/>
+        <origin xyz="0 0 -0.26" rpy="0 0 0"/>
+        <axis xyz="0 1 0"/>
+        <limit lower="-1.571" upper="1.571" effort="10.0" velocity="2.0"/>
+        <dynamics damping="0.3" friction="0.05"/>
+    </joint>
+    <!-- Gripper (parallel-jaw style, modeled as two finger pads + a palm) -->
+    <!-- Palm -->
+    <link name="right_gripper_palm">
     <visual>
       <geometry>
@@ -377,12 +417,12 @@
                ixy="0" ixz="0" iyz="0"/>
     </inertial>
-  </link>
-  <joint name="right_gripper_palm_joint" type="fixed">
-    <parent link="right_wrist_link"/>
-    <child link="right_gripper_palm"/>
-    <origin xyz="0 0 -0.025" rpy="0 0 0"/>
-  </joint>
-  <!-- Left Finger -->
-  <link name="right_gripper_left_finger">
+    </link>
+    <joint name="right_gripper_palm_joint" type="fixed">
+        <parent link="right_wrist_link"/>
+        <child link="right_gripper_palm"/>
+        <origin xyz="0 0 -0.025" rpy="0 0 0"/>
+    </joint>
+    <!-- Left Finger -->
+    <link name="right_gripper_left_finger">
     <visual>
       <geometry>
@@ -404,15 +444,15 @@
                ixy="0" ixz="0" iyz="0"/>
     </inertial>
-  </link>
-  <joint name="right_gripper_left_finger_joint" type="prismatic">
-    <parent link="right_gripper_palm"/>
-    <child link="right_gripper_left_finger"/>
-    <origin xyz="0 0.035 -0.01" rpy="0 0 0"/>
-    <axis xyz="0 1 0"/>
-    <limit lower="0.0" upper="0.02" effort="5.0" velocity="0.5"/>
-    <dynamics damping="0.2" friction="0.05"/>
-  </joint>
-  <!-- Right Finger -->
-  <link name="right_gripper_right_finger">
+    </link>
+    <joint name="right_gripper_left_finger_joint" type="prismatic">
+        <parent link="right_gripper_palm"/>
+        <child link="right_gripper_left_finger"/>
+        <origin xyz="0 0.035 -0.01" rpy="0 0 0"/>
+        <axis xyz="0 1 0"/>
+        <limit lower="0.0" upper="0.02" effort="5.0" velocity="0.5"/>
+        <dynamics damping="0.2" friction="0.05"/>
+    </joint>
+    <!-- Right Finger -->
+    <link name="right_gripper_right_finger">
     <visual>
       <geometry>
@@ -433,16 +473,16 @@
       <inertia ixx="0.0000175" iyy="0.0000154" izz="0.0000042"
                ixy="0" ixz="0" iyz="0"/>
-    </inertial>
-  </link>
-  <joint name="right_gripper_right_finger_joint" type="prismatic">
-    <parent link="right_gripper_palm"/>
-    <child link="right_gripper_right_finger"/>
-    <origin xyz="0 -0.035 -0.01" rpy="0 0 0"/>
-    <axis xyz="0 -1 0"/>
-    <limit lower="0.0" upper="0.02" effort="5.0" velocity="0.5"/>
-    <dynamics damping="0.2" friction="0.05"/>
-  </joint>
-  <!--  LEFT ARM (cosmetic / static — mirrors right arm visually)    -->
-  <link name="left_shoulder_link">
+        </inertial>
+    </link>
+    <joint name="right_gripper_right_finger_joint" type="prismatic">
+        <parent link="right_gripper_palm"/>
+        <child link="right_gripper_right_finger"/>
+        <origin xyz="0 -0.035 -0.01" rpy="0 0 0"/>
+        <axis xyz="0 -1 0"/>
+        <limit lower="0.0" upper="0.02" effort="5.0" velocity="0.5"/>
+        <dynamics damping="0.2" friction="0.05"/>
+    </joint>
+    <!--  LEFT ARM (cosmetic / static — mirrors right arm visually)    -->
+    <link name="left_shoulder_link">
     <visual>
       <geometry>
@@ -461,11 +501,11 @@
                ixy="0" ixz="0" iyz="0"/>
     </inertial>
-  </link>
-  <joint name="left_shoulder_joint" type="fixed">
-    <parent link="torso_link"/>
-    <child link="left_shoulder_link"/>
-    <origin xyz="0.0 0.12 0.48" rpy="0 0 0"/>
-  </joint>
-  <link name="left_upper_arm_link">
+    </link>
+    <joint name="left_shoulder_joint" type="fixed">
+        <parent link="torso_link"/>
+        <child link="left_shoulder_link"/>
+        <origin xyz="0.0 0.12 0.48" rpy="0 0 0"/>
+    </joint>
+    <link name="left_upper_arm_link">
     <visual>
       <geometry>
@@ -487,11 +527,11 @@
                ixy="0" ixz="0" iyz="0"/>
     </inertial>
-  </link>
-  <joint name="left_upper_arm_joint" type="fixed">
-    <parent link="left_shoulder_link"/>
-    <child link="left_upper_arm_link"/>
-    <origin xyz="0 0 0" rpy="0 0 0"/>
-  </joint>
-  <link name="left_elbow_link">
+    </link>
+    <joint name="left_upper_arm_joint" type="fixed">
+        <parent link="left_shoulder_link"/>
+        <child link="left_upper_arm_link"/>
+        <origin xyz="0 0 0" rpy="0 0 0"/>
+    </joint>
+    <link name="left_elbow_link">
     <visual>
       <geometry>
@@ -510,11 +550,11 @@
                ixy="0" ixz="0" iyz="0"/>
     </inertial>
-  </link>
-  <joint name="left_elbow_joint" type="fixed">
-    <parent link="left_upper_arm_link"/>
-    <child link="left_elbow_link"/>
-    <origin xyz="0 0 -0.28" rpy="0 0.5 0"/>
-  </joint>
-  <link name="left_forearm_link">
+    </link>
+    <joint name="left_elbow_joint" type="fixed">
+        <parent link="left_upper_arm_link"/>
+        <child link="left_elbow_link"/>
+        <origin xyz="0 0 -0.28" rpy="0 -1.5708 0"/>
+    </joint>
+    <link name="left_forearm_link">
     <visual>
       <geometry>
@@ -536,11 +576,11 @@
                ixy="0" ixz="0" iyz="0"/>
     </inertial>
-  </link>
-  <joint name="left_forearm_joint" type="fixed">
-    <parent link="left_elbow_link"/>
-    <child link="left_forearm_link"/>
-    <origin xyz="0 0 0" rpy="0 0 0"/>
-  </joint>
-  <link name="left_hand_link">
+    </link>
+    <joint name="left_forearm_joint" type="fixed">
+        <parent link="left_elbow_link"/>
+        <child link="left_forearm_link"/>
+        <origin xyz="0 0 0" rpy="0 0 0"/>
+    </joint>
+    <link name="left_hand_link">
     <visual>
       <geometry>
@@ -565,3 +605,188 @@
         <origin xyz="0 0 -0.28" rpy="0 0 0"/>
     </joint>
+    <!--  CAMERA — mounted on front of torso (not head)-->
+    <link name="camera_link">
+    <visual>
+      <geometry>
+        <box size="0.03 0.06 0.03"/>
+      </geometry>
+      <material name="black"/>
+    </visual>
+    <collision>
+      <geometry>
+        <box size="0.03 0.06 0.03"/>
+      </geometry>
+    </collision>
+    <inertial>
+      <mass value="0.1"/>
+      <inertia ixx="0.0000375" iyy="0.0000150" izz="0.0000375"
+               ixy="0" ixz="0" iyz="0"/>
+    </inertial>
+    </link>
+    <joint name="camera_joint" type="fixed">
+        <parent link="torso_link"/>
+        <child link="camera_link"/>
+        <!-- Front face of torso, roughly mid-height -->
+        <origin xyz="0.115 0 0.35" rpy="0 0 0"/>
+    </joint>
+    <!-- Camera optical frame (ROS convention: z forward, x right, y down) -->
+    <link name="camera_optical_frame"/>
+    <joint name="camera_optical_joint" type="fixed">
+        <parent link="camera_link"/>
+        <child link="camera_optical_frame"/>
+        <origin xyz="0 0 0" rpy="-1.5708 0 -1.5708"/>
+    </joint>
+    <!--  LIDAR — 2D scanning LiDAR on top of base, front              -->
+    <link name="lidar_link">
+        <visual>
+        <geometry>
+            <cylinder radius="0.04" length="0.04"/>
+        </geometry>
+        <material name="black"/>
+        </visual>
+        <collision>
+        <geometry>
+            <cylinder radius="0.04" length="0.04"/>
+        </geometry>
+        </collision>
+        <inertial>
+        <mass value="0.2"/>
+        <inertia ixx="0.0000453" iyy="0.0000453" izz="0.000160"
+                ixy="0" ixz="0" iyz="0"/>
+        </inertial>
+    </link>
+    <joint name="lidar_joint" type="fixed">
+        <parent link="base_link"/>
+        <child link="lidar_link"/>
+        <!-- Mounted on top of the base plate, front-center -->
+        <origin xyz="0.18 0 0.14" rpy="0 0 0"/>
+    </joint>
+    <!-- ============================================================ -->
+    <!--  GAZEBO PLUGINS  (Gazebo Harmonic / gz-sim)                   -->
+    <!-- ============================================================ -->
+    <gazebo>
+        <!-- Skid-steer drive controller -->
+        <plugin filename="gz-sim-diff-drive-system" name="gz::sim::systems::DiffDrive">
+            <left_joint>front_left_wheel_joint</left_joint>
+            <left_joint>rear_left_wheel_joint</left_joint>
+            <right_joint>front_right_wheel_joint</right_joint>
+            <right_joint>rear_right_wheel_joint</right_joint>
+            <wheel_separation>0.44</wheel_separation>
+            <wheel_radius>0.075</wheel_radius>
+            <max_linear_acceleration>1.0</max_linear_acceleration>
+            <max_angular_acceleration>2.0</max_angular_acceleration>
+            <topic>/cmd_vel</topic>
+            <odom_topic>/odom</odom_topic>
+            <tf_topic>/tf</tf_topic>
+            <frame_id>odom</frame_id>
+            <child_frame_id>base_footprint</child_frame_id>
+            <odom_publish_frequency>50</odom_publish_frequency>
+        </plugin>
+        <!-- Joint position controller for arm -->
+        <plugin filename="gz-sim-joint-position-controller-system"
+                name="gz::sim::systems::JointPositionController">
+            <joint_name>right_shoulder_joint</joint_name>
+            <topic>/right_shoulder_joint/cmd</topic>
+            <p_gain>30.0</p_gain>
+            <i_gain>0.1</i_gain>
+            <d_gain>5.0</d_gain>
+        </plugin>
+        <plugin filename="gz-sim-joint-position-controller-system"
+                name="gz::sim::systems::JointPositionController">
+            <joint_name>right_elbow_joint</joint_name>
+            <topic>/right_elbow_joint/cmd</topic>
+            <p_gain>20.0</p_gain>
+            <i_gain>0.1</i_gain>
+            <d_gain>3.0</d_gain>
+        </plugin>
+        <plugin filename="gz-sim-joint-position-controller-system"
+                name="gz::sim::systems::JointPositionController">
+            <joint_name>right_wrist_joint</joint_name>
+            <topic>/right_wrist_joint/cmd</topic>
+            <p_gain>10.0</p_gain>
+            <i_gain>0.05</i_gain>
+            <d_gain>2.0</d_gain>
+        </plugin>
+        <plugin filename="gz-sim-joint-position-controller-system"
+                name="gz::sim::systems::JointPositionController">
+            <joint_name>right_gripper_left_finger_joint</joint_name>
+            <topic>/right_gripper_left_finger_joint/cmd</topic>
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